File: AM4096q breakout.sch (KiCad schematic (older format))
At the start: 9 parts, among them IC1 AM4096Q, J1 Conn_01x03, J2 Conn_01x04, J3 Conn_01x04

Commit message: Added magnet presence LED
Parts:
- added D1: LED, LEDs:LED_0805, symbol Device:LED
- added R4: 51K, Resistors_SMD:R_0805, symbol Device:R
- C1: symbol CP -> Device:CP
- C2: symbol C -> Device:C
- IC1: symbol AM4096Q -> am4096q:AM4096Q
- J1: symbol Conn_01x03 -> conn:Conn_01x03
- J2, J3: symbol Conn_01x04 -> conn:Conn_01x04
- R1, R2, R3: symbol R -> Device:R
Connections:
- wire segments 9 -> 15
Changed lines of the file:
@@
-EESchema Schematic File Version 2
-LIBS:power
-LIBS:device
-LIBS:transistors
-LIBS:conn
-LIBS:linear
-LIBS:regul
-LIBS:74xx
-LIBS:cmos4000
-LIBS:adc-dac
-LIBS:memory
-LIBS:xilinx
-LIBS:microcontrollers
-LIBS:dsp
-LIBS:microchip
-LIBS:analog_switches
-LIBS:motorola
-LIBS:texas
-LIBS:intel
-LIBS:audio
-LIBS:interface
-LIBS:digital-audio
-LIBS:philips
-LIBS:display
-LIBS:cypress
-LIBS:siliconi
-LIBS:opto
-LIBS:atmel
-LIBS:contrib
-LIBS:valves
-LIBS:am4096q
-EELAYER 25 0
+EESchema Schematic File Version 4
+LIBS:AM4096q breakout-cache
+EELAYER 26 0
 EELAYER END
 $Descr A4 11693 8268
@@
 $EndDescr
 $Comp
-L AM4096Q IC1
+L am4096q:AM4096Q IC1
 U 1 1 5B21400D
 P 3400 3350
@@
 $EndComp
 $Comp
-L Conn_01x03 J1
+L conn:Conn_01x03 J1
 U 1 1 5B214054
 P 7350 1100
@@
 $EndComp
 $Comp
-L Conn_01x04 J2
+L conn:Conn_01x04 J2
 U 1 1 5B21407F
 P 7350 1700
@@
 $EndComp
 $Comp
-L Conn_01x04 J3
+L conn:Conn_01x04 J3
 U 1 1 5B2140A8
 P 7350 2450
@@
 $EndComp
 Wire Wire Line
-	7250 1300 7250 2650
+	7250 1300 7250 1900
 Connection ~ 7250 1900
 $Comp
-L GND #PWR01
+L power:GND #PWR01
 U 1 1 5B214139
 P 7250 2650
@@
 	1    0    0    -1
 $EndComp
-Wire Wire Line
-	7350 1300 7350 1900
-Wire Wire Line
-	7350 1850 7350 3450
-Connection ~ 7350 1850
 Connection ~ 7350 2650
 $Comp
-L R R1
+L Device:R R1
 U 1 1 5B2141B2
 P 2350 3300
@@
 VIN
 $Comp
-L R R2
+L Device:R R2
 U 1 1 5B21427C
 P 2350 3600
@@
 VIN
 $Comp
-L R R3
+L Device:R R3
 U 1 1 5B21429B
 P 2350 3700
@@
 AOUT
 $Comp
-L CP C1
+L Device:CP C1
 U 1 1 5B2143F8
 P 7150 3550
@@
 $EndComp
 $Comp
-L C C2
+L Device:C C2
 U 1 1 5B21443E
 P 7150 3800
@@
 	7350 3450 7300 3450
 Wire Wire Line
-	7300 3450 7300 3800
+	7300 3450 7300 3550
 Connection ~ 7300 3550
 Wire Wire Line
-	7000 3550 7000 3800
-$Comp
-L GND #PWR02
+	7000 3550 7000 3700
+$Comp
+L power:GND #PWR02
 U 1 1 5B2144C8
 P 7000 3700
@@
 	0    1    1    0
 $EndComp
-Connection ~ 10700 2900
 Connection ~ 7000 3700
 Text GLabel 7300 3800 3    60   Input ~ 0
@@
 VIN
 $Comp
-L GND #PWR03
+L power:GND #PWR03
 U 1 1 5B2146B2
 P 3450 2700
@@
 $EndComp
 $Comp
-L GND #PWR04
+L power:GND #PWR04
 U 1 1 5B2146E4
 P 3350 2700
@@
 $EndComp
 $Comp
-L GND #PWR05
+L power:GND #PWR05
 U 1 1 5B214716
 P 3250 2700
@@
 A
 $Comp
-L GND #PWR06
+L power:GND #PWR06
 U 1 1 5B214F3A
 P 4350 2850
@@
 	0    -1   -1   0
 $EndComp
+Wire Wire Line
+	7250 1900 7250 2650
+Wire Wire Line
+	7350 2650 7350 3450
+Wire Wire Line
+	7300 3550 7300 3800
+Wire Wire Line
+	7000 3700 7000 3800
+$Comp
+L Device:LED D1
+U 1 1 5B61D225
+P 3050 2250
+F 0 "D1" H 3042 1995 50  0000 C CNN
+F 1 "LED" H 3042 2086 50  0000 C CNN
+F 2 "LEDs:LED_0805" H 3050 2250 50  0001 C CNN
+F 3 "~" H 3050 2250 50  0001 C CNN
+	1    3050 2250
+	0    1    1    0
+$EndComp
+$Comp
+L Device:R R4
+U 1 1 5B61D37B
+P 3050 1900
+F 0 "R4" V 3130 1900 50  0000 C CNN
+F 1 "51K" V 3050 1900 50  0000 C CNN
+F 2 "Resistors_SMD:R_0805" V 2980 1900 50  0001 C CNN
+F 3 "" H 3050 1900 50  0001 C CNN
+	1    3050 1900
+	1    0    0    -1
+$EndComp
+$Comp
+L power:GND #PWR0101
+U 1 1 5B61D890
+P 3050 1650
+F 0 "#PWR0101" H 3050 1400 50  0001 C CNN
+F 1 "GND" H 3050 1500 50  0000 C CNN
+F 2 "" H 3050 1650 50  0001 C CNN
+F 3 "" H 3050 1650 50  0001 C CNN
+	1    3050 1650
+	-1   0    0    1
+$EndComp
+Wire Wire Line
+	3050 1650 3050 1750
+Wire Wire Line
+	7350 1300 7350 2650
+Wire Wire Line
+	3050 2050 3050 2100
+Wire Wire Line
+	3050 2700 3050 2400
 $EndSCHEMATC
